Commit message: new skeleton

File: io_mocap/description/blender_human_skeleton.urdf (robot description, URDF)
Before this commit: robot converted, 239 links, 238 joints
Links:
- removed link camera_color_optical_frame
- removed link link_Head_P
- removed link link_Head_R
- removed link link_Head_Y
- removed link link_Hips_P
- removed link link_Hips_R
- removed link link_Hips_Y
- removed link link_LeftArm_P
- removed link link_LeftArm_R
- removed link link_LeftArm_Y
- removed link link_LeftFoot_P
- removed link link_LeftFoot_R
- removed link link_LeftFoot_Y
- removed link link_LeftForeArm_P
- removed link link_LeftForeArm_R
- removed link link_LeftForeArm_Y
- removed link link_LeftHandIndex1_P
- removed link link_LeftHandIndex1_R
- removed link link_LeftHandIndex1_Y
- removed link link_LeftHandIndex2_P
- removed link link_LeftHandIndex2_R
- removed link link_LeftHandIndex2_Y
- removed link link_LeftHandIndex3_P
- removed link link_LeftHandIndex3_R
- removed link link_LeftHandIndex3_Y
- removed link link_LeftHandMiddle1_P
- removed link link_LeftHandMiddle1_R
- removed link link_LeftHandMiddle1_Y
- removed link link_LeftHandMiddle2_P
- removed link link_LeftHandMiddle2_R
- removed link link_LeftHandMiddle2_Y
- removed link link_LeftHandMiddle3_P
- removed link link_LeftHandMiddle3_R
- removed link link_LeftHandMiddle3_Y
- removed link link_LeftHandPinky1_P
- removed link link_LeftHandPinky1_R
- removed link link_LeftHandPinky1_Y
- removed link link_LeftHandPinky2_P
- removed link link_LeftHandPinky2_R
- removed link link_LeftHandPinky2_Y
- removed link link_LeftHandPinky3_P
- removed link link_LeftHandPinky3_R
- removed link link_LeftHandPinky3_Y
- removed link link_LeftHandRing1_P
- removed link link_LeftHandRing1_R
- removed link link_LeftHandRing1_Y
- removed link link_LeftHandRing2_P
- removed link link_LeftHandRing2_R
- removed link link_LeftHandRing2_Y
- removed link link_LeftHandRing3_P
- removed link link_LeftHandRing3_R
- removed link link_LeftHandRing3_Y
- removed link link_LeftHandThumb1_P
- removed link link_LeftHandThumb1_R
- removed link link_LeftHandThumb1_Y
- removed link link_LeftHandThumb2_P
- removed link link_LeftHandThumb2_R
- removed link link_LeftHandThumb2_Y
- removed link link_LeftHandThumb3_P
- removed link link_LeftHandThumb3_R
- removed link link_LeftHandThumb3_Y
- removed link link_LeftHand_P
- removed link link_LeftHand_R
- removed link link_LeftHand_Y
- removed link link_LeftInHandIndex_P
- removed link link_LeftInHandIndex_R
- removed link link_LeftInHandIndex_Y
- removed link link_LeftInHandMiddle_P
- removed link link_LeftInHandMiddle_R
- removed link link_LeftInHandMiddle_Y
- removed link link_LeftInHandPinky_P
- removed link link_LeftInHandPinky_R
- removed link link_LeftInHandPinky_Y
- removed link link_LeftInHandRing_P
- removed link link_LeftInHandRing_R
- removed link link_LeftInHandRing_Y
- removed link link_LeftLeg_P
- removed link link_LeftLeg_R
- removed link link_LeftLeg_Y
- removed link link_LeftShoulder_P
- removed link link_LeftShoulder_R
- removed link link_LeftShoulder_Y
- removed link link_LeftUpLeg_P
- removed link link_LeftUpLeg_R
- removed link link_LeftUpLeg_Y
- removed link link_Neck1_P
- removed link link_Neck1_R
- removed link link_Neck1_Y
- removed link link_Neck_P
- removed link link_Neck_R
- removed link link_Neck_Y
- removed link link_RightArm_P
- removed link link_RightArm_R
- removed link link_RightArm_Y
- removed link link_RightFoot_P
- removed link link_RightFoot_R
- removed link link_RightFoot_Y
- removed link link_RightForeArm_P
- removed link link_RightForeArm_R
- removed link link_RightForeArm_Y
- removed link link_RightHandIndex1_P
- removed link link_RightHandIndex1_R
- removed link link_RightHandIndex1_Y
- removed link link_RightHandIndex2_P
- removed link link_RightHandIndex2_R
- removed link link_RightHandIndex2_Y
- removed link link_RightHandIndex3_P
- removed link link_RightHandIndex3_R
- removed link link_RightHandIndex3_Y
- removed link link_RightHandMiddle1_P
- removed link link_RightHandMiddle1_R
- removed link link_RightHandMiddle1_Y
- removed link link_RightHandMiddle2_P
- removed link link_RightHandMiddle2_R
- removed link link_RightHandMiddle2_Y
- removed link link_RightHandMiddle3_P
- removed link link_RightHandMiddle3_R
- removed link link_RightHandMiddle3_Y
- removed link link_RightHandPinky1_P
- removed link link_RightHandPinky1_R
- removed link link_RightHandPinky1_Y
- removed link link_RightHandPinky2_P
- removed link link_RightHandPinky2_R
- removed link link_RightHandPinky2_Y
- removed link link_RightHandPinky3_P
- removed link link_RightHandPinky3_R
- removed link link_RightHandPinky3_Y
- removed link link_RightHandRing1_P
- removed link link_RightHandRing1_R
- removed link link_RightHandRing1_Y
- removed link link_RightHandRing2_P
- removed link link_RightHandRing2_R
- removed link link_RightHandRing2_Y
- removed link link_RightHandRing3_P
- removed link link_RightHandRing3_R
- removed link link_RightHandRing3_Y
- removed link link_RightHandThumb1_P
- removed link link_RightHandThumb1_R
- removed link link_RightHandThumb1_Y
- removed link link_RightHandThumb2_P
- removed link link_RightHandThumb2_R
- removed link link_RightHandThumb2_Y
- removed link link_RightHandThumb3_P
- removed link link_RightHandThumb3_R
- removed link link_RightHandThumb3_Y
- removed link link_RightHand_P
- removed link link_RightHand_R
- removed link link_RightHand_Y
- removed link link_RightInHandIndex_P
- removed link link_RightInHandIndex_R
- removed link link_RightInHandIndex_Y
- removed link link_RightInHandMiddle_P
- removed link link_RightInHandMiddle_R
- removed link link_RightInHandMiddle_Y
- removed link link_RightInHandPinky_P
- removed link link_RightInHandPinky_R
- removed link link_RightInHandPinky_Y
- removed link link_RightInHandRing_P
- removed link link_RightInHandRing_R
- removed link link_RightInHandRing_Y
- removed link link_RightLeg_P
- removed link link_RightLeg_R
- removed link link_RightLeg_Y
- removed link link_RightShoulder_P
- removed link link_RightShoulder_R
- removed link link_RightShoulder_Y
- removed link link_RightUpLeg_P
- removed link link_RightUpLeg_R
- removed link link_RightUpLeg_Y
- removed link link_Spine1_P
- removed link link_Spine1_R
- removed link link_Spine1_Y
- removed link link_Spine2_P
- removed link link_Spine2_R
- removed link link_Spine2_Y
- removed link link_Spine_P
- removed link link_Spine_R
- removed link link_Spine_Y
- link link_LeftSkeletonBase: mass 0.0665694383287888 -> 0.0381033782864806
- link link_LeftSkeletonIndex1: mass 0.00101710748996665 -> 0.00142104752116292
- link link_LeftSkeletonIndex2: mass 0.0074371750261936 -> 0.00558495597861908
- link link_LeftSkeletonIndex3: mass 0.0158610985851529 -> 0.00663689292635733
- link link_LeftSkeletonIndex4: mass 0.00285451442045608 -> 0.00283813624759799
- link link_LeftSkeletonMiddle1: mass 0.00101710748996666 -> 0.00142104751099454
- link link_LeftSkeletonMiddle2: mass 0.00743717502619359 -> 0.00558495571115789
- link link_LeftSkeletonMiddle3: mass 0.0158610985851528 -> 0.00663681790738949
- link link_LeftSkeletonMiddle4: mass 0.00285451142065185 -> 0.00283814024815753
- link link_LeftSkeletonPinky1: mass 0.00101710748996666 -> 0.00142104749852734
- link link_LeftSkeletonPinky2: mass 0.00743717502619359 -> 0.00558495640568594
- link link_LeftSkeletonPinky3: mass 0.0158610985851529 -> 0.00663681351825927
- link link_LeftSkeletonPinky4: mass 0.00285451773511369 -> 0.00283813750198794
- link link_LeftSkeletonRing1: mass 0.00101710748996666 -> 0.00142104751099453
- link link_LeftSkeletonRing2: mass 0.00743717502619359 -> 0.00558495571115816
- link link_LeftSkeletonRing3: mass 0.0158610985851529 -> 0.00663681790738944
- link link_LeftSkeletonRing4: mass 0.00285451142065188 -> 0.00283814024815758
- link link_LeftSkeletonThumb1: mass 0.00101710748996665 -> 0.00142104750359472
- link link_LeftSkeletonThumb2: mass 0.00826129582139841 -> 0.00619479805127877
- link link_LeftSkeletonThumb3: mass 0.0085937407191672 -> 0.00375708785451946
- link link_LeftSkeletonThumb4: mass 0.00285450549073411 -> 0.00283813885886545
- link link_LeftSkeletonThumbBase: mass 0.122473901434199 -> 0.00503517796554752
- link link_RightSkeletonBase: mass 0.0710882631261556 -> 0.0381015295019329
- link link_RightSkeletonIndex1: mass 0.00101710748996665 -> 0.00142104749535094
- link link_RightSkeletonIndex2: mass 0.00743717502619359 -> 0.00558495756330841
- link link_RightSkeletonIndex3: mass 0.0158610985851528 -> 0.00663685611795157
- link link_RightSkeletonIndex4: mass 0.00285451921524571 -> 0.00283814206573991
- link link_RightSkeletonMiddle1: mass 0.00101710748996666 -> 0.00142104751859945
- link link_RightSkeletonMiddle2: mass 0.0074371750261936 -> 0.00558495686016827
- link link_RightSkeletonMiddle3: mass 0.0158610985851529 -> 0.00663684957658263
- link link_RightSkeletonMiddle4: mass 0.00285451138566072 -> 0.00283813730192772
- link link_RightSkeletonPinky1: mass 0.00101710748996666 -> 0.00142104752949724
- link link_RightSkeletonPinky2: mass 0.00743717502619359 -> 0.0055849572264132
- link link_RightSkeletonPinky3: mass 0.0158610985851529 -> 0.00663684736422184
- link link_RightSkeletonPinky4: mass 0.00285451193827601 -> 0.0028381369220279
- link link_RightSkeletonRing1: mass 0.00101710748996665 -> 0.00142104751859945
- link link_RightSkeletonRing2: mass 0.00743717502619358 -> 0.00558495686016845
- link link_RightSkeletonRing3: mass 0.0158610985851528 -> 0.00663684971073181
- link link_RightSkeletonRing4: mass 0.00285451138566076 -> 0.00283813730192769
- link link_RightSkeletonThumb1: mass 0.00101710748996665 -> 0.00142104750359472
- link link_RightSkeletonThumb2: mass 0.00826129582139841 -> 0.00619479805127885
- link link_RightSkeletonThumb3: mass 0.0085937407191672 -> 0.00375708793059457
- link link_RightSkeletonThumb4: mass 0.0028545054907341 -> 0.00283813885886545
- link link_RightSkeletonThumbBase: mass 0.117950008013029 -> 0.00503517876942867
Joints:
- removed joint joint_Head_Camera
- removed joint joint_Head_P
- removed joint joint_Head_R
- removed joint joint_Head_Y
- removed joint joint_Hips_P
- removed joint joint_Hips_R
- removed joint joint_Hips_Y
- removed joint joint_LeftArm_P
- removed joint joint_LeftArm_R
- removed joint joint_LeftArm_Y
- removed joint joint_LeftFoot_P
- removed joint joint_LeftFoot_R
- removed joint joint_LeftFoot_Y
- removed joint joint_LeftForeArm_P
- removed joint joint_LeftForeArm_R
- removed joint joint_LeftForeArm_Y
- removed joint joint_LeftHandIndex1_P
- removed joint joint_LeftHandIndex1_R
- removed joint joint_LeftHandIndex1_Y
- removed joint joint_LeftHandIndex2_P
- removed joint joint_LeftHandIndex2_R
- removed joint joint_LeftHandIndex2_Y
- removed joint joint_LeftHandIndex3_P
- removed joint joint_LeftHandIndex3_R
- removed joint joint_LeftHandIndex3_Y
- removed joint joint_LeftHandMiddle1_P
- removed joint joint_LeftHandMiddle1_R
- removed joint joint_LeftHandMiddle1_Y
- removed joint joint_LeftHandMiddle2_P
- removed joint joint_LeftHandMiddle2_R
- removed joint joint_LeftHandMiddle2_Y
- removed joint joint_LeftHandMiddle3_P
- removed joint joint_LeftHandMiddle3_R
- removed joint joint_LeftHandMiddle3_Y
- removed joint joint_LeftHandPinky1_P
- removed joint joint_LeftHandPinky1_R
- removed joint joint_LeftHandPinky1_Y
- removed joint joint_LeftHandPinky2_P
- removed joint joint_LeftHandPinky2_R
- removed joint joint_LeftHandPinky2_Y
- removed joint joint_LeftHandPinky3_P
- removed joint joint_LeftHandPinky3_R
- removed joint joint_LeftHandPinky3_Y
- removed joint joint_LeftHandRing1_P
- removed joint joint_LeftHandRing1_R
- removed joint joint_LeftHandRing1_Y
- removed joint joint_LeftHandRing2_P
- removed joint joint_LeftHandRing2_R
- removed joint joint_LeftHandRing2_Y
- removed joint joint_LeftHandRing3_P
- removed joint joint_LeftHandRing3_R
- removed joint joint_LeftHandRing3_Y
- removed joint joint_LeftHandThumb1_P
- removed joint joint_LeftHandThumb1_R
- removed joint joint_LeftHandThumb1_Y
- removed joint joint_LeftHandThumb2_P
- removed joint joint_LeftHandThumb2_R
- removed joint joint_LeftHandThumb2_Y
- removed joint joint_LeftHandThumb3_P
- removed joint joint_LeftHandThumb3_R
- removed joint joint_LeftHandThumb3_Y
- removed joint joint_LeftHand_P
- removed joint joint_LeftHand_R
- removed joint joint_LeftHand_Y
- removed joint joint_LeftInHandIndex_P
- removed joint joint_LeftInHandIndex_R
- removed joint joint_LeftInHandIndex_Y
- removed joint joint_LeftInHandMiddle_P
- removed joint joint_LeftInHandMiddle_R
- removed joint joint_LeftInHandMiddle_Y
- removed joint joint_LeftInHandPinky_P
- removed joint joint_LeftInHandPinky_R
- removed joint joint_LeftInHandPinky_Y
- removed joint joint_LeftInHandRing_P
- removed joint joint_LeftInHandRing_R
- removed joint joint_LeftInHandRing_Y
- removed joint joint_LeftLeg_P
- removed joint joint_LeftLeg_R
- removed joint joint_LeftLeg_Y
- removed joint joint_LeftShoulder_P
- removed joint joint_LeftShoulder_R
- removed joint joint_LeftShoulder_Y
- removed joint joint_LeftUpLeg_P
- removed joint joint_LeftUpLeg_R
- removed joint joint_LeftUpLeg_Y
- removed joint joint_Neck1_P
- removed joint joint_Neck1_R
- removed joint joint_Neck1_Y
- removed joint joint_Neck_P
- removed joint joint_Neck_R
- removed joint joint_Neck_Y
- removed joint joint_RightArm_P
- removed joint joint_RightArm_R
- removed joint joint_RightArm_Y
- removed joint joint_RightFoot_P
- removed joint joint_RightFoot_R
- removed joint joint_RightFoot_Y
- removed joint joint_RightForeArm_P
- removed joint joint_RightForeArm_R
- removed joint joint_RightForeArm_Y
- removed joint joint_RightHandIndex1_P
- removed joint joint_RightHandIndex1_R
- removed joint joint_RightHandIndex1_Y
- removed joint joint_RightHandIndex2_P
- removed joint joint_RightHandIndex2_R
- removed joint joint_RightHandIndex2_Y
- removed joint joint_RightHandIndex3_P
- removed joint joint_RightHandIndex3_R
- removed joint joint_RightHandIndex3_Y
- removed joint joint_RightHandMiddle1_P
- removed joint joint_RightHandMiddle1_R
- removed joint joint_RightHandMiddle1_Y
- removed joint joint_RightHandMiddle2_P
- removed joint joint_RightHandMiddle2_R
- removed joint joint_RightHandMiddle2_Y
- removed joint joint_RightHandMiddle3_P
- removed joint joint_RightHandMiddle3_R
- removed joint joint_RightHandMiddle3_Y
- removed joint joint_RightHandPinky1_P
- removed joint joint_RightHandPinky1_R
- removed joint joint_RightHandPinky1_Y
- removed joint joint_RightHandPinky2_P
- removed joint joint_RightHandPinky2_R
- removed joint joint_RightHandPinky2_Y
- removed joint joint_RightHandPinky3_P
- removed joint joint_RightHandPinky3_R
- removed joint joint_RightHandPinky3_Y
- removed joint joint_RightHandRing1_P
- removed joint joint_RightHandRing1_R
- removed joint joint_RightHandRing1_Y
- removed joint joint_RightHandRing2_P
- removed joint joint_RightHandRing2_R
- removed joint joint_RightHandRing2_Y
- removed joint joint_RightHandRing3_P
- removed joint joint_RightHandRing3_R
- removed joint joint_RightHandRing3_Y
- removed joint joint_RightHandThumb1_P
- removed joint joint_RightHandThumb1_R
- removed joint joint_RightHandThumb1_Y
- removed joint joint_RightHandThumb2_P
- removed joint joint_RightHandThumb2_R
- removed joint joint_RightHandThumb2_Y
- removed joint joint_RightHandThumb3_P
- removed joint joint_RightHandThumb3_R
- removed joint joint_RightHandThumb3_Y
- removed joint joint_RightHand_P
- removed joint joint_RightHand_R
- removed joint joint_RightHand_Y
- removed joint joint_RightInHandIndex_P
- removed joint joint_RightInHandIndex_R
- removed joint joint_RightInHandIndex_Y
- removed joint joint_RightInHandMiddle_P
- removed joint joint_RightInHandMiddle_R
- removed joint joint_RightInHandMiddle_Y
- removed joint joint_RightInHandPinky_P
- removed joint joint_RightInHandPinky_R
- removed joint joint_RightInHandPinky_Y
- removed joint joint_RightInHandRing_P
- removed joint joint_RightInHandRing_R
- removed joint joint_RightInHandRing_Y
- removed joint joint_RightLeg_P
- removed joint joint_RightLeg_R
- removed joint joint_RightLeg_Y
- removed joint joint_RightShoulder_P
- removed joint joint_RightShoulder_R
- removed joint joint_RightShoulder_Y
- removed joint joint_RightUpLeg_P
- removed joint joint_RightUpLeg_R
- removed joint joint_RightUpLeg_Y
- removed joint joint_Spine1_P
- removed joint joint_Spine1_R
- removed joint joint_Spine1_Y
- removed joint joint_Spine2_P
- removed joint joint_Spine2_R
- removed joint joint_Spine2_Y
- removed joint joint_Spine_P
- removed joint joint_Spine_R
- removed joint joint_Spine_Y
- joint joint_LeftSkeletonBase: axis 0 1 0 -> (none); limit lower=-3.1415926536 upper=3.1415926536 effort=100.0000 velocity=3.0000 -> (none); origin xyz=-0.02 0 -0.1 rpy=-1.5707963268 0 1.5707963268 -> xyz=-0.05 0 0 rpy=0 0 0; parent link_LeftHand_Y -> base_link
- joint joint_LeftSkeletonIndex1: origin xyz=0.022 0.0026506 -0.0019547 rpy=-0.023349 0.26078 0.029576 -> xyz=0.021871 0.0026351 -0.0024377 rpy=0 0.2618 0.1199
- joint joint_LeftSkeletonIndex2: origin xyz=0.0026 0.0062204 0.0071414 rpy=-0.75647 0 0 -> xyz=0.0036 0.0074761 0.0074414 rpy=-0.75647 0 0
- joint joint_LeftSkeletonIndex3: origin xyz=0 0.043889 0.062046 rpy=-0.81433 0 0 -> xyz=0 0.043889 0.062046 rpy=0.46849 0 0
- joint joint_LeftSkeletonIndex4: origin xyz=0 0.031696 0.067973 rpy=1.7453 0 0 -> xyz=0 0.064952 0.0375 rpy=1.2217 0 0
- joint joint_LeftSkeletonMiddle1: origin xyz=0 0 0.001 rpy=0 0 0.1199 -> xyz=0 0 0.0005 rpy=0 0 0.1199
- joint joint_LeftSkeletonMiddle2: origin xyz=0.0026 0.0062204 0.0071414 rpy=-0.75647 0 0 -> xyz=0.0036 0.0074761 0.0074414 rpy=-0.75647 0 0
- joint joint_LeftSkeletonMiddle3: origin xyz=0 0.043889 0.062046 rpy=-0.81433 0 0 -> xyz=0 0.043889 0.062046 rpy=0.46849 0 0
- joint joint_LeftSkeletonMiddle4: origin xyz=0 0.031696 0.067973 rpy=1.7453 0 0 -> xyz=0 0.064952 0.0375 rpy=1.2217 0 0
- joint joint_LeftSkeletonPinky1: origin xyz=-0.0431 -0.0051927 -0.0013494 rpy=-0.015367 -0.17386 0.20851 -> xyz=-0.042036 -0.0050645 -0.0016681 rpy=0 -0.17453 0.1199
- joint joint_LeftSkeletonPinky2: origin xyz=0.0026 0.0062204 0.0071414 rpy=-0.75647 0 0 -> xyz=0.0036 0.0074761 0.0074414 rpy=-0.75647 0 0
- joint joint_LeftSkeletonPinky3: origin xyz=0 0.043889 0.062046 rpy=-0.81433 0 0 -> xyz=0 0.043889 0.062046 rpy=0.46849 0 0
- joint joint_LeftSkeletonPinky4: origin xyz=0 0.031696 0.067973 rpy=1.7453 0 0 -> xyz=0 0.064952 0.0375 rpy=1.2217 0 0
- joint joint_LeftSkeletonRing1: origin xyz=-0.020849 -0.002512 0.001 rpy=0 0 0.1199 -> xyz=-0.020849 -0.002512 0.0005 rpy=0 0 0.1199
- joint joint_LeftSkeletonRing2: origin xyz=0.0026 0.0062204 0.0071414 rpy=-0.75647 0 0 -> xyz=0.0036 0.0074761 0.0074414 rpy=-0.75647 0 0
- joint joint_LeftSkeletonRing3: origin xyz=0 0.043889 0.062046 rpy=-0.81433 0 0 -> xyz=0 0.043889 0.062046 rpy=0.46849 0 0
- joint joint_LeftSkeletonRing4: origin xyz=0 0.031696 0.067973 rpy=1.7453 0 0 -> xyz=0 0.064952 0.0375 rpy=1.2217 0 0
- joint joint_LeftSkeletonThumb1: origin xyz=0.0085 -0.006 0.01972 rpy=1.5708 -1.5708 0 -> xyz=-0.0072 -0.006 -0.0195 rpy=1.5708 1.5708 0
- joint joint_LeftSkeletonThumb2: origin xyz=0.0026 0.0062204 0.0071414 rpy=-1.1345 0 0 -> xyz=0.0036 0.0074761 0.0074414 rpy=-1.309 0 0
- joint joint_LeftSkeletonThumbBase: axis -1 0 0 -> 1 0 0; origin xyz=0.040994 -0.053404 -0.015 rpy=-3.1416 0 -2.1405 -> xyz=0.040042 -0.053331 -0.015 rpy=0 0 0.99442
- joint joint_RightSkeletonBase: axis 0 1 0 -> (none); limit lower=-3.1415926536 upper=3.1415926536 effort=100.0000 velocity=3.0000 -> (none); origin xyz=0.02 0 -0.1 rpy=-1.5707963268 0 -1.5707963268 -> xyz=0.05 0 0 rpy=0 0 0; parent link_RightHand_Y -> base_link
- joint joint_RightSkeletonIndex1: origin xyz=-0.022 0.0026506 -0.0019547 rpy=-0.023349 -0.26078 -0.029576 -> xyz=-0.021871 0.0026351 -0.0024377 rpy=0 -0.2618 -0.1199
- joint joint_RightSkeletonIndex2: origin xyz=0.0026 0.0062204 0.0071414 rpy=-0.75647 0 0 -> xyz=0.0036 0.0074761 0.0074414 rpy=-0.75647 0 0
- joint joint_RightSkeletonIndex3: origin xyz=0 0.043889 0.062046 rpy=-0.81433 0 0 -> xyz=0 0.043889 0.062046 rpy=0.46849 0 0
- joint joint_RightSkeletonIndex4: origin xyz=0 0.031696 0.067973 rpy=1.7453 0 0 -> xyz=0 0.064952 0.0375 rpy=1.2217 0 0
- joint joint_RightSkeletonMiddle1: origin xyz=0 0 0.001 rpy=0 0 -0.1199 -> xyz=0 0 0.0005 rpy=0 0 -0.1199
- joint joint_RightSkeletonMiddle2: origin xyz=0.0026 0.0062204 0.0071414 rpy=-0.75647 0 0 -> xyz=0.0036 0.0074761 0.0074414 rpy=-0.75647 0 0
- joint joint_RightSkeletonMiddle3: origin xyz=0 0.043889 0.062046 rpy=-0.81433 0 0 -> xyz=0 0.043889 0.062046 rpy=0.46849 0 0
- joint joint_RightSkeletonMiddle4: origin xyz=0 0.031696 0.067973 rpy=1.7453 0 0 -> xyz=0 0.062616 0.040744 rpy=1.2217 0 0
- joint joint_RightSkeletonPinky1: origin xyz=0.0431 -0.0051927 -0.0013494 rpy=-0.015367 0.17386 -0.20851 -> xyz=0.042036 -0.0050645 -0.0016681 rpy=0 0.17453 -0.1199
- joint joint_RightSkeletonPinky2: origin xyz=0.0026 0.0062204 0.0071414 rpy=-0.75647 0 0 -> xyz=0.0036 0.0074761 0.0074414 rpy=-0.75647 0 0
- joint joint_RightSkeletonPinky3: origin xyz=0 0.043889 0.062046 rpy=-0.81433 0 0 -> xyz=0 0.043889 0.062046 rpy=0.46849 0 0
- joint joint_RightSkeletonPinky4: origin xyz=0 0.031696 0.067973 rpy=1.7453 0 0 -> xyz=0 0.064952 0.0375 rpy=1.2217 0 0
- joint joint_RightSkeletonRing1: origin xyz=0.020849 -0.002512 0.001 rpy=0 0 -0.1199 -> xyz=0.020849 -0.002512 0.0005 rpy=0 0 -0.1199
- joint joint_RightSkeletonRing2: origin xyz=0.0026 0.0062204 0.0071414 rpy=-0.75647 0 0 -> xyz=0.0036 0.0074761 0.0074414 rpy=-0.75647 0 0
- joint joint_RightSkeletonRing3: origin xyz=0 0.043889 0.062046 rpy=-0.81433 0 0 -> xyz=0 0.043889 0.062046 rpy=0.46849 0 0
- joint joint_RightSkeletonRing4: origin xyz=0 0.031696 0.067973 rpy=1.7453 0 0 -> xyz=0 0.062616 0.040744 rpy=1.2217 0 0
- joint joint_RightSkeletonThumb1: origin xyz=-0.0085 -0.006 0.01972 rpy=1.5708 1.5708 0 -> xyz=-0.0072 -0.006 0.0195 rpy=1.5708 1.5708 0
- joint joint_RightSkeletonThumb2: origin xyz=0.0026 0.0062204 0.0071414 rpy=-1.1345 0 0 -> xyz=0.0036 0.0074761 0.0074414 rpy=-1.309 0 0
- joint joint_RightSkeletonThumbBase: origin xyz=-0.040994 -0.053404 -0.015 rpy=-3.1416 0 2.1405 -> xyz=-0.040042 -0.053331 -0.015 rpy=3.1416 0 2.1472
