Commit message: update v4 urdf

File: io_mocap/description/blender_human_skeleton_v4.urdf (robot description, URDF)
Before this commit: robot skeleton_hands, 61 links, 60 joints
Links:
- link link_LeftSkeletonBase: mass 0.0381033782864806 -> 0.052266
- link link_LeftSkeletonIndex1: mass 0.00142104752116292 -> 0.00180132347270952
- link link_LeftSkeletonIndex2: mass 0.00558495597861908 -> 0.00674975819974668
- link link_LeftSkeletonIndex3: mass 0.00663689292635733 -> 0.009553
- link link_LeftSkeletonMiddle1: mass 0.00142104751099454 -> 0.00180132346254114
- link link_LeftSkeletonMiddle2: mass 0.00558495571115789 -> 0.00674975793228549
- link link_LeftSkeletonMiddle3: mass 0.00663681790738949 -> 0.00955296694624449
- link link_LeftSkeletonMiddle4: mass 0.00283814024815753 -> 0.0028381
- link link_LeftSkeletonPinky1: mass 0.00142104749852734 -> 0.00180132345007395
- link link_LeftSkeletonPinky2: mass 0.00558495640568594 -> 0.00674975862681354
- link link_LeftSkeletonPinky3: mass 0.00663681351825927 -> 0.00955296255386165
- link link_LeftSkeletonRing1: mass 0.00142104751099453 -> 0.00180132346254114
- link link_LeftSkeletonRing2: mass 0.00558495571115816 -> 0.0067498
- link link_LeftSkeletonRing3: mass 0.00663681790738944 -> 0.00955296694624447
- link link_LeftSkeletonThumb2: mass 0.00619479805127877 -> 0.00750354561222259
- link link_LeftSkeletonThumb3: mass 0.00375708785451946 -> 0.00507456373320865
- link link_LeftSkeletonThumbBase: mass 0.00503517796554752 -> 0.0050352
- link link_RightSkeletonBase: mass 0.0381015295019329 -> 0.0518268058409403
- link link_RightSkeletonIndex1: mass 0.00142104749535094 -> 0.0018013
- link link_RightSkeletonIndex2: mass 0.00558495756330841 -> 0.0067498
- link link_RightSkeletonIndex3: mass 0.00663685611795157 -> 0.009553
- link link_RightSkeletonIndex4: mass 0.00283814206573991 -> 0.0028381
- link link_RightSkeletonMiddle1: mass 0.00142104751859945 -> 0.0018013
- link link_RightSkeletonMiddle2: mass 0.00558495686016827 -> 0.0067498
- link link_RightSkeletonMiddle3: mass 0.00663684957658263 -> 0.009553
- link link_RightSkeletonMiddle4: mass 0.00283813730192772 -> 0.0028381
- link link_RightSkeletonPinky1: mass 0.00142104752949724 -> 0.00180132348104385
- link link_RightSkeletonPinky2: mass 0.0055849572264132 -> 0.0067498
- link link_RightSkeletonPinky3: mass 0.00663684736422184 -> 0.009553
- link link_RightSkeletonPinky4: mass 0.0028381369220279 -> 0.0028381
- link link_RightSkeletonRing1: mass 0.00142104751859945 -> 0.0018013
- link link_RightSkeletonRing2: mass 0.00558495686016845 -> 0.0067498
- link link_RightSkeletonRing3: mass 0.00663684971073181 -> 0.009553
- link link_RightSkeletonRing4: mass 0.00283813730192769 -> 0.0028381
- link link_RightSkeletonThumb1: mass 0.00142104750359472 -> 0.001421
- link link_RightSkeletonThumb2: mass 0.00619479805127885 -> 0.00750354561222267
- link link_RightSkeletonThumb3: mass 0.00375708793059457 -> 0.00507456380928375
- link link_RightSkeletonThumb4: mass 0.00283813885886545 -> 0.0028381
- link link_RightSkeletonThumbBase: mass 0.00503517876942867 -> 0.0050352
Joints:
- joint joint_RightSkeletonMiddle4: origin xyz=0 0.062616 0.040744 rpy=1.2217 0 0 -> xyz=0 0.064952 0.0375 rpy=1.2217 0 0
- joint joint_RightSkeletonRing4: origin xyz=0 0.062616 0.040744 rpy=1.2217 0 0 -> xyz=0 0.064952 0.0375 rpy=1.2217 0 0
- joint joint_RightSkeletonThumb4: limit lower=0 upper=0 effort=0 velocity=0 -> lower=-3.14 upper=3.14 effort=100 velocity=1
